File: KiCAD_files/ADB-3020-CDV.sch (KiCad schematic (older format))
At the start: 115 parts, among them IC1 7812T, IC2 NE5532N, IC3 LM2576, IC4 NE555, IC5 IR2184D, J1 + IN, J2 - IN, J3 + OUT, J4 - OUT, J5 + IN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

Commit message: Removed all ERC, repaired annotation on sch and pcb, added sheet pcb info, revisited .sch component name value position
Parts:
- B1: symbol D_Bridge_+A-A -> D_Bridge_+A-A-RESCUE-ADB-3020-CDV
- renumbered FAN41 to FAN1, FAULT41 to FAULT1, HEAT41 to HEAT1, LIMITER41 to LIMITER1, ON41 to ON1
Other:
- note added: "± Shunt"
- note removed: "~ Shunt"
